File: hardware/BaseBoard.sch (EAGLE design)
At the start: 10 parts

Commit message: Layout and route base board
Connections:
- new net !JNTRST!: U$6.P14
- new net !NRST!: U$6.P15, U$7.P12
- new net A01: U$1.P16, U$8.A16
- new net A02: U$1.P17, U$8.A17
- new net A03: U$1.P18, U$8.A18
- new net A04: U$1.P19, U$8.A19
- new net A05: U$1.P20, U$8.A20
- new net A06: U$1.P21, U$8.A21
- new net A07: U$1.P22, U$8.A22
- new net A08: U$1.P23, U$8.B16
- new net A09: U$1.P24, U$8.B17
- new net A10: U$1.P25, U$8.B18
- new net A11: U$1.P26, U$8.B19
- new net A12: U$1.P27, U$8.B20
- new net A13: U$1.P28, U$8.B21
- new net A14: U$1.P29, U$8.B22
- new net A15: U$1.P30, U$8.B23
- new net B01: U$2.P16, U$8.A26
- new net B02: U$2.P17, U$8.A27
- new net B03: U$2.P18, U$8.A28
- new net B04: U$2.P19, U$8.A29
- new net B05: U$2.P20, U$8.A30
- new net B06: U$2.P21, U$8.A31
- new net B07: U$2.P22, U$8.A32
- new net B08: U$2.P23, U$8.B26
- new net B09: U$2.P24, U$8.B27
- new net B10: U$2.P25, U$8.B28
- new net B11: U$2.P26, U$8.B29
- new net B12: U$2.P27, U$8.B30
- new net B13: U$2.P28, U$8.B31
- new net B14: U$2.P29, U$8.B32
- new net B15: U$2.P30, U$8.B33
- new net C01: U$3.P16, U$8.A36
- new net C02: U$3.P17, U$8.A37
- new net C03: U$3.P18, U$8.A38
- new net C04: U$3.P19, U$8.A39
- new net C05: U$3.P20, U$8.A40
- new net C06: U$3.P21, U$8.A41
- new net C07: U$3.P22, U$8.A42
- new net C08: U$3.P23, U$8.B36
- new net C09: U$3.P24, U$8.B37
- new net C10: U$3.P25, U$8.B38
- new net C11: U$3.P26, U$8.B39
- new net C12: U$3.P27, U$8.B40
- new net C13: U$3.P28, U$8.B41
- new net C14: U$3.P29, U$8.B42
- new net C15: U$3.P30, U$8.B43
- new net CANH: CN1.3, CN2.3, U$1.P7, U$2.P7, U$3.P7, U$4.P7, U$5.P7, U$6.P7
- new net CANL: CN1.2, CN2.2, U$1.P6, U$2.P6, U$3.P6, U$4.P6, U$5.P6, U$6.P6
- new net D01: U$4.P16, U$8.A46
- new net D02: U$4.P17, U$8.A47
- new net D03: U$4.P18, U$8.A48
- new net D04: U$4.P19, U$8.A49
- new net D05: U$4.P20, U$8.A50
- new net D06: U$4.P21, U$8.A51
- new net D07: U$4.P22, U$8.A52
- new net D08: U$4.P23, U$8.B46
- new net D09: U$4.P24, U$8.B47
- new net D10: U$4.P25, U$8.B48
- new net D11: U$4.P26, U$8.B49
- new net D12: U$4.P27, U$8.B50
- new net D13: U$4.P28, U$8.B51
- new net D14: U$4.P29, U$8.B52
- new net D15: U$4.P30, U$8.B53
- new net E01: U$5.P16, U$8.A56
- new net E02: U$5.P17, U$8.A57
- new net E03: U$5.P18, U$8.A58
- new net E04: U$5.P19, U$8.A59
- new net E05: U$5.P20, U$8.A60
- new net E06: U$5.P21, U$8.A61
- new net E07: U$5.P22, U$8.A62
- new net E08: U$5.P23, U$8.B56
- new net E09: U$5.P24, U$8.B57
- new net E10: U$5.P25, U$8.B58
- new net E11: U$5.P26, U$8.B59
- new net E12: U$5.P27, U$8.B60
- new net E13: U$5.P28, U$8.B61
- new net E14: U$5.P29, U$8.B62
- new net E15: U$5.P30, U$8.B63
- new net F01: U$6.P16, U$8.A66
- new net F02: U$6.P17, U$8.A67
- new net F03: U$6.P18, U$8.A68
- new net F04: U$6.P19, U$8.A69
- new net F05: U$6.P20, U$8.A70
- new net F06: U$6.P21, U$8.A71
- new net F07: U$6.P22, U$8.A72
- new net F08: U$6.P23, U$8.B66
- new net F09: U$6.P24, U$8.B67
- new net F10: U$6.P25, U$8.B68
- new net F11: U$6.P26, U$8.B69
- new net F12: U$6.P27, U$8.B70
- new net F13: U$6.P28, U$8.B71
- new net F14: U$6.P29, U$8.B72
- new net F15: U$6.P30, U$8.B73
- new net GND: CN1.4, CN2.4, U$1.P5, U$1.P8, U$2.P5, U$2.P8, U$3.P5, U$3.P8, U$4.P5, U$4.P8, U$5.P5, U$5.P8, U$6.P5, U$6.P8, U$7.P11, U$7.P5, U$7.P7, U$8.A12, U$8.A13, U$8.A14, U$8.A15, U$8.A23, U$8.A24, U$8.A25, U$8.A33, U$8.A34, U$8.A35, U$8.A43, U$8.A44, U$8.A45, U$8.A53, U$8.A54, U$8.A55, U$8.A63, U$8.A64, U$8.A65, U$8.B12, U$8.B13, U$8.B14, U$8.B15, U$8.B24, U$8.B25, U$8.B34, U$8.B35, U$8.B44, U$8.B45, U$8.B54, U$8.B55, U$8.B64, U$8.B65
- new net JCLK: U$7.P9
- new net JCLK/SWCLK: U$6.P11, U$7.P6
- new net JTDI: U$6.P12, U$7.P10
- new net JTDO/SWO: U$6.P13, U$7.P8
- new net JTMS/SWDIO: U$6.P10, U$7.P4
- new net N$11: U$1.P10
- new net N$118: U$5.P10
- new net N$119: U$5.P11
- new net N$12: U$1.P11
- new net N$120: U$5.P12
- new net N$121: U$5.P13
- new net N$122: U$5.P14
- new net N$123: U$5.P15
- new net N$13: U$1.P12
- new net N$14: U$1.P13
- new net N$15: U$1.P14
- new net N$16: U$1.P15
- new net N$180: U$8.B74
- new net N$181: U$8.B75
- new net N$191: U$8.B76
- new net N$192: U$8.B77
- new net N$193: U$8.B78
- new net N$194: U$8.B79
- new net N$195: U$8.B80
- new net N$196: U$8.B81
- new net N$197: U$8.B82
- new net N$259: U$8.A73
- new net N$260: U$8.A74
- new net N$262: U$8.A75
- new net N$263: U$8.A76
- new net N$264: U$8.A77
- new net N$265: U$8.A78
- new net N$266: U$8.A79
- new net N$267: U$8.A80
- new net N$268: U$8.A81
- new net N$269: U$8.A82
- new net N$3: U$2.P10
- new net N$4: U$2.P11
- new net N$5: U$2.P12
- new net N$6: U$2.P13
- new net N$60: U$3.P10
- new net N$61: U$3.P11
- new net N$62: U$3.P12
- new net N$63: U$3.P13
- new net N$64: U$3.P14
- new net N$65: U$3.P15
- new net N$7: U$2.P14
- new net N$8: U$2.P15
- new net N$89: U$4.P10
- new net N$90: U$4.P11
- new net N$91: U$4.P12
- new net N$92: U$4.P13
- new net N$93: U$4.P14
- new net N$94: U$4.P15
- new net T_VCC: U$7.P3
- new net VBU: U$1.P4, U$2.P4, U$3.P4, U$4.P4, U$5.P4, U$6.P4
- new net VCC: U$1.P2, U$2.P2, U$3.P2, U$4.P2, U$5.P2, U$6.P2
- new net VCP_RX: U$7.P13
- new net VCP_TX: U$7.P14
- new net VDD: U$1.P3, U$2.P3, U$3.P3, U$4.P3, U$5.P3, U$6.P3
- new net VPP: CN1.1, CN2.1, U$1.P1, U$2.P1, U$3.P1, U$4.P1, U$5.P1, U$6.P1
Other:
- moved on the sheet: CN1, CN2, U$2, U$3, U$4, U$5, U$6, U$7, U$8

Commit message: Complete base board
Parts:
- renumbered U$1 to A, U$2 to B, U$3 to C, U$4 to D, U$5 to E, U$6 to F
