File: hardware/sensing.brd (EAGLE design)
At the start: 47 x 40.5 mm, 52 parts

Commit message: Clean silk print
Other:
- board text added: "Designed by @fujiy0, 2019"
- board text added: "Sensing & GPIO Module"
Changed lines of the file:
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@@
 <grid distance="50" unitdist="mil" unit="mm" style="dots" multiple="1" display="yes" altdistance="5" altunitdist="mil" altunit="mm"/>
 <layers>
-<layer number="1" name="Top" color="4" fill="1" visible="yes" active="yes"/>
+<layer number="1" name="Top" color="4" fill="1" visible="no" active="yes"/>
 <layer number="2" name="Route2" color="16" fill="1" visible="no" active="no"/>
 <layer number="3" name="Route3" color="17" fill="1" visible="no" active="no"/>
@@
 <layer number="28" name="bValues" color="7" fill="1" visible="no" active="yes"/>
 <layer number="29" name="tStop" color="7" fill="3" visible="no" active="yes"/>
-<layer number="30" name="bStop" color="7" fill="6" visible="no" active="yes"/>
+<layer number="30" name="bStop" color="7" fill="6" visible="yes" active="yes"/>
 <layer number="31" name="tCream" color="7" fill="4" visible="no" active="yes"/>
 <layer number="32" name="bCream" color="7" fill="5" visible="no" active="yes"/>
@@
 <hole x="54" y="-17.25" drill="2.6"/>
 <hole x="54" y="17.25" drill="2.6"/>
-<text x="54.61" y="0" size="1.9304" layer="29" font="vector" rot="R90" align="center">WASA Rocket Project</text>
-<text x="54.61" y="0" size="1.9304" layer="1" font="vector" rot="R90" align="center">WASA Rocket Project</text>
+<text x="54.61" y="0" size="2.1844" layer="29" font="vector" ratio="9" rot="R90" align="center">WASA Rocket Project</text>
+<text x="54.61" y="0" size="2.1844" layer="1" font="vector" rot="R90" align="center">WASA Rocket Project</text>
+<text x="12.065" y="0" size="1.27" layer="25" font="vector" rot="R90" align="center">Sensing &amp; GPIO Module</text>
+<text x="55.88" y="-7.62" size="0.8128" layer="30" font="vector" rot="MR270" align="center">Designed by @fujiy0, 2019</text>
+<polygon width="0" layer="21">
+<vertex x="10.16" y="17.78"/>
+<vertex x="11.43" y="18.542"/>
+<vertex x="11.43" y="17.018"/>
+</polygon>
 </plain>
 <attributes>
@@
 </element>
 <element name="CA" library="jst-ph" package="S2B-PH-K-S" value="" x="34.29" y="16.51" smashed="yes">
-<attribute name="NAME" x="31.29" y="23.51" size="0.8128" layer="25" font="vector" ratio="10"/>
+<attribute name="NAME" x="34.338" y="14.62" size="1.27" layer="25" font="vector" ratio="10" align="center"/>
 <attribute name="VALUE" x="31.29" y="12.51" size="1.27" layer="27"/>
 </element>
 <element name="SA" library="jst-ph" package="S3B-PH-K-S" value="" x="15.875" y="16.51" smashed="yes">
-<attribute name="NAME" x="15.685" y="14.62" size="0.8128" layer="25" font="vector" ratio="10"/>
+<attribute name="NAME" x="15.939" y="14.62" size="1.27" layer="25" font="vector" ratio="10" align="center"/>
 <attribute name="VALUE" x="11.875" y="12.51" size="1.27" layer="27"/>
 </element>
 <element name="SB" library="jst-ph" package="S3B-PH-K-S" value="" x="25.654" y="16.51" smashed="yes">
-<attribute name="NAME" x="21.654" y="23.51" size="0.8128" layer="25" font="vector" ratio="10"/>
+<attribute name="NAME" x="25.718" y="14.62" size="1.27" layer="25" font="vector" ratio="10" align="center"/>
 <attribute name="VALUE" x="21.654" y="12.51" size="1.27" layer="27"/>
 </element>
@@
 </element>
 <element name="CB" library="jst-ph" package="S2B-PH-K-S" value="" x="41.91" y="16.51" smashed="yes">
-<attribute name="NAME" x="38.91" y="23.51" size="0.8128" layer="25" font="vector" ratio="10"/>
+<attribute name="NAME" x="41.958" y="14.62" size="1.27" layer="25" font="vector" ratio="10" align="center"/>
 <attribute name="VALUE" x="38.91" y="12.51" size="1.27" layer="27"/>
 </element>
