File: hardware/USB&LiPoPower.sch (EAGLE design)
At the start: 48 parts, among them Q1 IRLML5203, Q2 IRLML5203, U2 ACS711ELCTR-12AB-T, U3 ACS711ELCTR-12AB-T, U4 I-02247_NJM2845, U5 CH004-2032LF

Commit message: Layout USB and LiPo power board
Parts:
- removed C1: 47µF, rcl:CPOL-EUE2.5-6
- removed C2: 22µF, rcl:CPOL-EUE2.5-5
- removed CL3, CL4: 15pF, rcl:C-EUC0603K
- removed FC-1: 32.768kHz, crystal':CRYTALFC-255
- removed PS1: HT7750A_SOT23-3, HT7750A_SOT23-3:HT7750A_SOT23-3
- removed Q1, Q2: IRLML5203, transistor-power:IRLML5203
- removed R_PROG: (no value), rcl:R-US_R0402
- removed S1: SSAJ120100, SSAJ120100:SSAJ120100
- removed U$5: MCP73831, mcp73831:MCP73831
- removed U$6: SK-12D01-VG4, switches:SK-12D01-VG4
- removed U4: I-02247_NJM2845, akizuki:I-02247_NJM2845
- removed U5: CH004-2032LF, CH004-2032LF:CH004-2032LF
- added 3.3V: I-02247_NJM2845, akizuki:I-02247_NJM2845
- added 5V: HT7750A_SOT23-3, HT7750A_SOT23-3:HT7750A_SOT23-3
- added BACKUP, POWER: SK-12D01-VG4, switches:SK-12D01-VG4
- added C16, C17: 47µF, rcl:CPOL-EUUD-5X5,8
- added CHARGER: MCP73831, mcp73831:MCP73831
- added D3, D4: RB160M-30TR, RB160M-30TR:RB160M-30TR
- added G1: CH291-1220LF, battery:CH291-1220LF
- added LIPO_SW, USB_SW, VCC_SEL, VPP_SEL: IRLML5203, transistor-power:IRLML5203
- added R3: 100k, rcl:R-US_R0603
- added RPROG: (no value), rcl:R-US_R0603
- R1: device rcl:R-US_R0402 -> rcl:R-US_R0603
Connections:
- net N$3 renamed 5VC_OUT
- net N$4 renamed 3.3VC_OUT
- removed net BU+: S1.1, U5.2
- removed net N$2: D1.A, PS1.LX, U$3.2
- removed net N$71: CL4.2, FC-1.1, STM32F001.PC15/OSC32_OUT
- removed net N$72: CL3.2, FC-1.2, STM32F001.PC14/OSC32_IN
- removed net VCC'1: C4.1, D2.K, Q2.S, U4.VIN
- new net BAT+: BACKUP.B, G1.+
- new net N$10: D3.K, D4.K, R3.2
- new net N$9: LIPO_SW.G, POWER.C, R3.1, USB_SW.G
- new net USB_5V: D4.A, U$1.VCC, USB_SW.S
- new net VBU: BACKUP.C, U$2.VBAT
- new net VCCG_IN: 5V.LX, D1.A, U$3.2
- net 3.3V: now also 3.3V.VOUT; no longer U4.VOUT
- net 5V: now also VCC_SEL.S; no longer Q1.S
- net GND: now also 3.3V.GND, 5V.GND, C16.-, C17.-, CHARGER.VSS, G1.-, POWER.A, RPROG.1, U$1.GND@1, U$1.GND@2; no longer C1.-, C2.-, CL3.1, CL4.1, PS1.GND, R_PROG.2, U$5.VSS, U4.GND, U5.1
- net LIPO+: now also CHARGER.VBAT, D3.A, LIPO_SW.S; no longer U$5.VBAT, U$6.C
- net N$1: now also CHARGER.PROG, RPROG.2; no longer R_PROG.1, U$5.PROG
- net VBAT: no longer S1.C, U$2.VBAT
- net VCC_GEN: now also 5V.VOUT, C17.+, VCC_SEL.D; no longer C2.+, PS1.VOUT, Q1.D
- net VCC_USB: now also CHARGER.VDD, USB_SW.D, VCC_SEL.G, VPP_SEL.G; no longer Q1.G, Q2.G, U$1.VCC, U$5.VDD
- net VLIPO: now also C16.+, LIPO_SW.D, VPP_SEL.D; no longer C1.+, Q2.D, U$6.B
- net VPP: now also 3.3V.VIN, C4.1, D2.K, VPP_SEL.S
Other:
- moved on the sheet: C14, C15, C3, C4, C5, C6, D, D1, D2, DA1.1, DA1.2, LIPO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

Commit message: Complete USB & LiPo power board
Parts:
- removed LED1: (no value), led:LEDCHIP-LED0603
- removed R: 1K, rcl:R-US_R0603
- added IC1, IC2: 4066D, 40xx:4066D
- added LED: (no value), led:LEDCHIP-LED0603
- added R10, R17: 10k, resistor:R-US_R0603
- added R11, R12, R13, R14, R15, R16, R18, R9: 1k, resistor:R-US_R0603
- added R2, R5, R6, R7, R8: 10k, rcl:R-US_R0603
- added R4: 1k, rcl:R-US_R0603
- added RLED: 1K, rcl:R-US_R0603
- C10, C11, C12, C5, C6, C7, C8, C9: value (none) -> 0.1µF
- renumbered 3.3V to IC4, 5V to IC3, D to D5, DA1 to OP, G1 to CR1201, LIPO_SW to T2, MCP1 to MCP2562, U$1 to MICRO_USB, U$3 to I, U2 to VCCC, U3 to VDDC, USB_SW to T1, VCC_SEL to T3, VPP_SEL to T4
Connections:
- removed net N$45: U$2.P8
- removed net N$46: U$2.P7
- removed net N$47: U$2.P6
- removed net N$48: U$2.P5
- removed net N$49: U$2.P4
- removed net N$50: U$2.P3
- removed net N$51: STM32F001.PA0/USART4_TX/WKUP1/ADC_IN0
- removed net N$52: STM32F001.PA1/ADC_IN1/COMP1_INP/USART4_RX
- removed net N$53: STM32F001.PA2/ADC_IN2/WKUP4USART2_TX
- removed net N$54: STM32F001.PA3/ADC_IN3/COMP2_INP/USART2_RX
- removed net N$55: STM32F001.PA4/ADC_IN4/DAC_OUT1
- removed net N$56: STM32F001.PA5/ADC_IN5/DAC_OUT2/SPI1_SCK
- removed net N$57: STM32F001.PA6/ADC_IN6/SPI1_MISO/TIM3_CH1
- removed net N$58: STM32F001.PA7/ADC_IN7/SPI1_MOSI/TIM3_CH2
- removed net N$59: STM32F001.PA8/TIM1_CH1
- removed net N$62: STM32F001.PB0/ADC_IN8/TIM3_CH3
- removed net N$63: STM32F001.PB1/ADC_IN9/TIM3_CH4
- removed net N$64: STM32F001.PB2
- removed net N$65: STM32F001.PB10/I2C2_SCL/TIM2_CH3/USART3_TX
- removed net N$66: STM32F001.PB11/I2C2_SDA/TIM2_C4/USART3_RX
- removed net N$67: STM32F001.PB12
- removed net N$68: STM32F001.PB13/SPI2_SCK/I2C2_SCL
- removed net N$69: STM32F001.PB14/SPI2_MISO/I2C2_SDA
- removed net N$70: STM32F001.PB15/WKUP7/RTC_REFIN/SPI2_MOSI
- removed net N$76: LED1.A, R.2
- removed net VBAT: STM32F001.VBATT(P1)
- new net !HIL!: IC1A.C, IC1B.C, IC2A.C, IC2B.C, IC2C.C, IC2D.C, R10.1, R9.1
- new net 3.3VC': IC1B.A, OP.2.OUT, RF2.2
- new net 3.3VC_OUT': RC2.1, VDDC.VOUT
- new net 5VC': IC1A.A, OP.1.OUT, RF1.2
- new net 5VC_OUT': RC1.1, VCCC.VOUT
- new net N$2: CHARGER.STAT, R17.2
- new net N$3: LED.C, RLED.1
- new net PVCC: IC2C.A, R5.1, R6.2
- new net PVDD: IC2D.A, R7.1, R8.2
- new net PVPP: IC2B.A, R2.1, R4.2
- new net STAT: R17.1, R18.1, STM32F001.PA1/ADC_IN1/COMP1_INP/USART4_RX
- new net SVBU: IC2A.B, R14.1, STM32F001.PA6/ADC_IN6/SPI1_MISO/TIM3_CH1
- new net SVCC: IC2C.B, R11.1, STM32F001.PB1/ADC_IN9/TIM3_CH4
- new net SVDD: IC2D.B, R12.1, STM32F001.PB0/ADC_IN8/TIM3_CH3
- new net SVPP: IC2B.B, R13.1, STM32F001.PA7/ADC_IN7/SPI1_MOSI/TIM3_CH2
- net 3.3V: now also R7.2
- net 3.3VC: now also IC1B.B, R15.1, STM32F001.PA5/ADC_IN5/DAC_OUT2/SPI1_SCK; no longer OP.2.OUT, RC2.1, RF2.2, VDDC.VOUT
- net 5V: now also R5.2
- net 5VC: now also IC1A.B, R16.1, STM32F001.PA4/ADC_IN4/DAC_OUT1; no longer OP.1.OUT, RC1.1, RF1.2, VCCC.VOUT
- net GND: now also R4.1, R6.1, R8.1
- net N$33: now also R16.2
- net N$34: now also R15.2
- net N$35: now also R14.2
- net N$36: now also R13.2
- net N$43: now also R12.2
- net N$44: now also R11.2
- net N$73: now also RLED.2, STM32F001.PC13/WKUP2/RTC_TAMP1/RTC_TS/RTC_OUT; no longer LED1.C, STM32F001.PA15/USART2_RX
- net N$74: now also R9.2
- net N$75: now also R18.2
- net VBU: now also IC2A.A, STM32F001.VBATT(P1)
- net VCC: now also LED.A
- net VDD: now also R10.2; no longer R.1
- net VPP: now also R2.2

Commit message: Some fixes
Parts:
- RPROG: value (none) -> 4.7k
Changed lines of the file:
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@@
 <part name="C16" library="rcl" library_urn="urn:adsk.eagle:library:334" deviceset="CPOL-EU" device="UD-5X5,8" package3d_urn="urn:adsk.eagle:package:23470/1" value="47µF"/>
 <part name="C17" library="rcl" library_urn="urn:adsk.eagle:library:334" deviceset="CPOL-EU" device="UD-5X5,8" package3d_urn="urn:adsk.eagle:package:23470/1" value="47µF"/>
-<part name="RPROG" library="rcl" library_urn="urn:adsk.eagle:library:334" deviceset="R-US_" device="R0603" package3d_urn="urn:adsk.eagle:package:23555/3"/>
+<part name="RPROG" library="rcl" library_urn="urn:adsk.eagle:library:334" deviceset="R-US_" device="R0603" package3d_urn="urn:adsk.eagle:package:23555/3" value="4.7k"/>
 <part name="R1" library="rcl" library_urn="urn:adsk.eagle:library:334" deviceset="R-US_" device="R0603" package3d_urn="urn:adsk.eagle:package:23555/3" value="10k"/>
 <part name="BACKUP" library="switches" deviceset="SK-12D01-VG4" device=""/>
