File: hardware/BatteryPowerV2.brd (EAGLE design)
At the start: 47 x 40.5 mm, 66 parts, among them Q1 IRLML6402, U1 LT1616ES6TRMPBF, U2 LT6106CS5#PBF, U3 LT1616ES6TRMPBF, U4 LT6106CS5#PBF, U5 TCK106AF,LF, U6 TCK106AF,LF

Commit message: 修正途中
Routing:
- net VCC: track 83.2 -> 82.1 mm
- net BAT1: track 13.8 -> 14.6 mm
