File: hardware/LoRa.brd (EAGLE design)
At the start: 47 x 40.5 mm, 26 parts, among them J1 U.FL-R-SMT, J2 U.FL-R-SMT, J3 U.FL-R-SMT, U1 E220-900T22S, U2 E220-900T22S

Commit message: LoRaモジュール、基板設計完了です。
Routing:
- net GND: track 208.5 -> 325.5 mm, vias 59 -> 54
- net LORA2_TRX: track 0.00 -> 71.7 mm, vias 0 -> 2
- net LORA2_RTX: track 0.00 -> 64.8 mm, vias 0 -> 2
- net VDD: track 71.9 -> 135.5 mm, vias 8 -> 12
- net LORA1_RTX: track 0.00 -> 56.6 mm, vias 0 -> 1
- net LORA1_TRX: track 0.00 -> 54.4 mm, vias 0 -> 1
- net LORA2_M0: track 0.00 -> 29.4 mm, vias 0 -> 1
- net LORA2_M1: track 0.00 -> 28.3 mm, vias 0 -> 1
- net N$6: track 0.00 -> 28.0 mm, vias 0 -> 2
- net LORA2_AUX: track 0.00 -> 25.0 mm, vias 0 -> 1
- net N$10: track 0.00 -> 20.7 mm, vias 0 -> 2
- net N$1: track 0.00 -> 17.4 mm, vias 0 -> 1
- net LORA1_M0: track 0.00 -> 15.4 mm, vias 0 -> 1
- net LORA1_M1: track 0.00 -> 14.3 mm, vias 0 -> 1
- net N$73: track 6.02 -> 20.2 mm, vias 0 -> 2
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
Commit message: 修正途中
Connections:
- removed net LORA_AUX: STM32F001.22
- net LORA1_AUX: now also STM32F001.22
Routing:
- net LORA1_AUX: track 0.00 -> 3.91 mm, vias 0 -> 1
Changed lines of the file:
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@@
 <signal name="LORA1_AUX">
 <contactref element="U1" pad="P9"/>
+<contactref element="STM32F001" pad="22"/>
+<wire x1="27.01" y1="-3.33" x2="29.238" y2="-3.33" width="0.254" layer="1"/>
+<wire x1="29.238" y1="-3.33" x2="29.337" y2="-3.429" width="0.254" layer="1"/>
+<via x="29.337" y="-3.429" extent="1-16" drill="0.35"/>
+<wire x1="29.337" y1="-3.429" x2="29.386" y2="-3.38" width="0.254" layer="16"/>
+<wire x1="29.386" y1="-3.38" x2="30.86" y2="-3.38" width="0.254" layer="16"/>
 </signal>
 <signal name="LORA2_M0">
@@
 <wire x1="27.94" y1="-18.415" x2="28.575" y2="-18.415" width="0.254" layer="1"/>
 </signal>
-<signal name="LORA_AUX">
-<contactref element="STM32F001" pad="22"/>
-</signal>
 </signals>
