File: hardware/LoRa.sch (EAGLE design)
At the start: 26 parts, among them J1 U.FL-R-SMT, J2 U.FL-R-SMT, J3 U.FL-R-SMT, U1 E220-900T22S, U2 E220-900T22S

Commit message: 修正途中
Connections:
- removed net LORA_AUX: STM32F001.PB11/I2C2_SDA/TIM2_C4/USART3_RX
- net LORA1_AUX: now also STM32F001.PB11/I2C2_SDA/TIM2_C4/USART3_RX
Changed lines of the file:
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@@
 <label x="264.16" y="96.52" size="1.778" layer="95" rot="R180" xref="yes"/>
+</segment>
+<segment>
+<pinref part="STM32F001" gate="G$1" pin="PB11/I2C2_SDA/TIM2_C4/USART3_RX"/>
+<wire x1="121.92" y1="25.4" x2="144.78" y2="25.4" width="0.1524" layer="91"/>
+<label x="144.78" y="25.4" size="1.778" layer="95" xref="yes"/>
 </segment>
 </net>
@@
 </segment>
 </net>
-<net name="LORA_AUX" class="0">
-<segment>
-<pinref part="STM32F001" gate="G$1" pin="PB11/I2C2_SDA/TIM2_C4/USART3_RX"/>
-<wire x1="121.92" y1="25.4" x2="144.78" y2="25.4" width="0.1524" layer="91"/>
-<label x="144.78" y="25.4" size="1.778" layer="95" xref="yes"/>
-</segment>
-</net>
